Commit message: Update arm.urdf.xacro

File: arm_ws/src/arm_description/urdf/arm.urdf.xacro (robot description, xacro)
@@ -33,5 +33,5 @@
         <parent link="base_link"/>
         <child link = "base_plate"/>
-        <origin xyz="0 0 0.307"/>
+        <origin xyz="0 0 0.307"/>   <!-- Distance image one -->
         <axis xyz="0 0 1"/>
         <limit lower="-${PI / 2}" upper="${PI / 2}"
@@ -51,5 +51,5 @@
         <parent link="base_plate"/>
         <child link = "forward_drive_arm"/>
-        <origin xyz="-0.02 0 0.35"/>
+        <origin xyz="-0.02 0 0.35"/> <!-- Distance image two-->
         <axis xyz="1 0 0"/>
         <limit lower="-${PI / 2}" upper="${PI / 2}"
@@ -68,5 +68,5 @@
         <parent link="forward_drive_arm"/>
         <child link = "horizontal_arm"/>
-        <origin xyz="0 0 0.8"/>
+        <origin xyz="0 0 0.8"/> <!-- Distance image three -->
         <axis xyz="1 0 0"/>
         <limit lower="-${PI / 2}" upper="${PI / 2}"
@@ -85,5 +85,5 @@
         <parent link="horizontal_arm"/>
         <child link = "claw_support"/>
-        <origin xyz="0 0.82 0"/>
+        <origin xyz="0 0.82 0"/> <!-- Distance image four-->
     </joint>
     <!-- Link  gripper -->
@@ -107,5 +107,5 @@
         <parent link="claw_support"/>
         <child link = "gripper_right"/>
-        <origin xyz="-0.04 0.13 -0.1"/>
+        <origin xyz="-0.04 0.13 -0.1"/> <!-- Distance image five -->
         <axis xyz="0 0 1"/>
         <limit lower="-${PI / 2}" upper="0.0"
@@ -115,5 +115,5 @@
         <parent link="claw_support"/>
         <child link = "gripper_left"/>
-        <origin xyz="-0.22 0.13 -0.1"/>
+        <origin xyz="-0.22 0.13 -0.1"/> <!-- Distance image five -->
         <axis xyz="0 0 1"/>
         <limit lower="0.0" upper="${PI / 2}"

Commit message: Version action task moveit

File: arm_ws/src/arm_description/urdf/arm.urdf.xacro (robot description, xacro)
@@ -1,11 +1,51 @@
 <?xml version="1.0"?>
 <robot xmlns:xacro="http://www.ros.org/wiki/xacro" name="arm">
-     <!-- Useful XACRO Variables (Properties) -->
-     <xacro:property name="PI" value="3.14159265359" />
-     <xacro:property name="effort" value="30.0" />
-     <xacro:property name="velocity" value="10.0" />
-    <!-- Links  base-->
+     <!-- Definir Materiales -->
+  <material name="red">
+    <color rgba="1 0 0 1"/>
+  </material>
+  <material name="blue">
+    <color rgba="0 0 1 1"/>
+  </material>
+  <material name="green">
+    <color rgba="0 1 0 1"/>
+  </material>
+  <material name="yellow">
+    <color rgba="1 1 0 1"/> <!-- Amarillo opaco -->
+  </material>
+  <material name="purple">
+    <color rgba="0.5 0 0.5 1"/> <!-- Púrpura opaco -->
+  </material>
+    <!-- Include Gazebo Parameters -->
+    <xacro:include filename="$(find arm_description)/urdf/arm_gazebo.xacro" />
+    <!-- Include ros2_control Plugins -->
+    <xacro:include filename="$(find arm_description)/urdf/arm_ros2_control.xacro" />
+    <!-- Useful XACRO Variables (Properties) -->
+    <xacro:property name="PI" value="3.14159265359" />
+    <xacro:property name="effort" value="30.0" />
+    <xacro:property name="velocity" value="10.0" />
+    <!-- Useful Macros -->
+    <xacro:macro name="default_inertial" params="mass">
+        <inertial>
+            <origin xyz="0 0 0" rpy="0 0 0"/>
+            <mass value="${mass}" />
+            <inertia ixx="1.0" ixy="0.0" ixz="0.0"
+                     iyy="1.0" iyz="0.0"
+                     izz="1.0" />
+        </inertial>
+    </xacro:macro>
+    <xacro:macro name="default_transmission" params="number">
+        <transmission name="transmission_${number}">
+            <plugin>transmission_interface/SimpleTransmission</plugin>
+            <actuator name="motor_${number}" role="actuator1"/>
+            <joint name="joint_${number}"    role="joint1">
+                <mechanical_reduction>1.0</mechanical_reduction>
+            </joint>
+        </transmission>
+    </xacro:macro>
+    <!-- Links -->
     <link name="world"/>
     <link name="base_link">
+        <xacro:default_inertial mass="1.0"/>
         <visual>
             <origin rpy="0 0 0" xyz="-0.5 -0.5 0"/>
@@ -13,107 +53,156 @@
                 <mesh filename="package://arm_description/meshes/basement.STL" scale="0.01 0.01 0.01"/>
             </geometry>
-        </visual>
-    </link>
-     <!-- Joint base_link -->
-     <joint name="virtual_joint" type="fixed">
+            <material name="blue"/>  <!-- Asignar color azul -->
+        </visual>
+        <collision>
+            <origin rpy="0 0 0" xyz="-0.5 -0.5 0"/>
+            <geometry>
+                <mesh filename="package://arm_description/meshes/basement.STL" scale="0.01 0.01 0.01"/>
+            </geometry>
+        </collision>
+    </link>
+    <link name="base_plate">
+        <xacro:default_inertial mass="0.1"/>
+        <visual>
+            <origin rpy="0 0 0" xyz="-0.39 -0.39 -0.56"/>
+            <geometry>
+                <mesh filename="package://arm_description/meshes/base_plate.STL" scale="0.01 0.01 0.01"/>
+            </geometry>
+            <material name="yellow"/>  <!-- Asignar color azul -->
+        </visual>
+        <collision>
+            <origin rpy="0 0 0" xyz="-0.39 -0.39 -0.56"/>
+            <geometry>
+                <mesh filename="package://arm_description/meshes/base_plate.STL" scale="0.01 0.01 0.01"/>
+            </geometry>
+        </collision>
+    </link>
+    <link name="forward_drive_arm">
+        <xacro:default_inertial mass="0.1"/>
+        <visual>
+            <origin rpy=" 0 -${PI / 2} ${PI / 2}" xyz="0.19 0.06 -0.08"/>
+            <geometry>
+                <mesh filename="package://arm_description/meshes/forward_drive_arm.STL" scale="0.01 0.01 0.01"/>
+            </geometry>
+            <material name="red"/>  <!-- Asignar color azul -->
+        </visual>
+        <collision>
+            <origin rpy=" 0 -${PI / 2} ${PI / 2}" xyz="0.19 0.06 -0.08"/>
+            <geometry>
+                <mesh filename="package://arm_description/meshes/forward_drive_arm.STL" scale="0.01 0.01 0.01"/>
+            </geometry>
+        </collision>
+    </link>
+    <link name="horizontal_arm">
+        <xacro:default_inertial mass="0.1"/>
+        <visual>
+            <origin rpy="${PI / 2} 0 ${PI / 2}" xyz="-0.03 -0.4 -0.06"/>
+            <geometry>
+                <mesh filename="package://arm_description/meshes/horizontal_arm.STL" scale="0.01 0.01 0.01"/>
+            </geometry>
+            <material name="red"/>  <!-- Asignar color azul -->
+        </visual>
+        <collision>
+            <origin rpy="${PI / 2} 0 ${PI / 2}" xyz="-0.03 -0.4 -0.06"/>
+            <geometry>
+                <mesh filename="package://arm_description/meshes/horizontal_arm.STL" scale="0.01 0.01 0.01"/>
+            </geometry>
+        </collision>
+    </link>
+    <link name="claw_support">
+        <xacro:default_inertial mass="0.05"/>
+        <visual>
+            <origin rpy="0 0 ${PI / 2}" xyz="0 -0.05 -0.15"/>
+            <geometry>
+                <mesh filename="package://arm_description/meshes/claw_support.STL" scale="0.01 0.01 0.01"/>
+            </geometry>
+            <material name="blue"/>  <!-- Asignar color azul -->
+        </visual>
+        <collision>
+            <origin rpy="0 0 ${PI / 2}" xyz="0 -0.05 -0.15"/>
+            <geometry>
+                <mesh filename="package://arm_description/meshes/claw_support.STL" scale="0.01 0.01 0.01"/>
+            </geometry>
+        </collision>
+    </link>
+    <link name="gripper_right">
+        <xacro:default_inertial mass="0.01"/>
+        <visual>
+            <origin rpy="0 0 -${PI / 2}" xyz="-0.1 0.50 -0.1"/>
+            <geometry>
+                <mesh filename="package://arm_description/meshes/right_finger.STL" scale="0.01 0.01 0.01"/>
+            </geometry>
+            <material name="green"/>  <!-- Asignar color azul -->
+        </visual>
+        <collision>
+            <origin rpy="0 0 -${PI / 2}" xyz="-0.1 0.50 -0.1"/>
+            <geometry>
+                <mesh filename="package://arm_description/meshes/right_finger.STL" scale="0.01 0.01 0.01"/>
+            </geometry>
+        </collision>
+    </link>
+    <link name="gripper_left">
+        <xacro:default_inertial mass="0.01"/>
+        <visual>
+            <origin rpy="0 0 -${PI / 2}" xyz="-0.04 0.50 -0.1"/>
+            <geometry>
+                <mesh filename="package://arm_description/meshes/left_finger.STL" scale="0.01 0.01 0.01"/>
+            </geometry>
+            <material name="green"/>  <!-- Asignar color azul -->
+        </visual>
+        <collision>
+            <origin rpy="0 0 -${PI / 2}" xyz="-0.04 0.50 -0.1"/>
+            <geometry>
+                <mesh filename="package://arm_description/meshes/left_finger.STL" scale="0.01 0.01 0.01"/>
+            </geometry>
+        </collision>
+    </link>
+    <!-- Joints -->
+    <joint name="virtual_joint" type="fixed">
         <parent link="world"/>
         <child link="base_link"/>
         <origin xyz="0 0 0" rpy="0 0 0"/>
     </joint>
-    <!-- Links  base plate-->
-    <link name="base_plate">
-        <visual>
-            <origin rpy="0 0 0" xyz="-0.39 -0.39 -0.56"/>
-            <geometry>
-                <mesh filename="package://arm_description/meshes/base_plate.STL" scale="0.01 0.01 0.01"/>
-            </geometry>
-        </visual>
-    </link>
     <joint name ="joint_1" type="revolute">
         <parent link="base_link"/>
         <child link = "base_plate"/>
-        <origin xyz="0 0 0.307"/>   <!-- Distance image one -->
+        <origin xyz="0 0 0.307"/>
         <axis xyz="0 0 1"/>
         <limit lower="-${PI / 2}" upper="${PI / 2}"
                effort="${effort}" velocity="${velocity}"/>
     </joint>
-    <!-- Links  brazo derecho-->
-    <link name="forward_drive_arm">
-        <visual>
-            <origin rpy=" 0 -${PI / 2} ${PI / 2}" xyz="0.19 0.06 -0.08"/>
-            <geometry>
-                <mesh filename="package://arm_description/meshes/forward_drive_arm.STL" scale="0.01 0.01 0.01"/>
-            </geometry>
-        </visual>
-    </link>
-     <!-- Joint 2 -->
-     <joint name ="joint_2" type="revolute">
+    <joint name ="joint_2" type="revolute">
         <parent link="base_plate"/>
         <child link = "forward_drive_arm"/>
-        <origin xyz="-0.02 0 0.35"/> <!-- Distance image two-->
+        <origin xyz="-0.02 0 0.35"/>
         <axis xyz="1 0 0"/>
         <limit lower="-${PI / 2}" upper="${PI / 2}"
                 effort="${effort}" velocity="${velocity}"/>
     </joint>
- <!-- Links  Horizontal arm-->
-    <link name="horizontal_arm">
-        <visual>
-            <origin rpy="${PI / 2} 0 ${PI / 2}" xyz="-0.03 -0.4 -0.06"/>
-            <geometry>
-                <mesh filename="package://arm_description/meshes/horizontal_arm.STL" scale="0.01 0.01 0.01"/>
-            </geometry>
-        </visual>
-    </link>
     <joint name ="joint_3" type="revolute">
         <parent link="forward_drive_arm"/>
         <child link = "horizontal_arm"/>
-        <origin xyz="0 0 0.8"/> <!-- Distance image three -->
+        <origin xyz="0 0 0.8"/>
         <axis xyz="1 0 0"/>
         <limit lower="-${PI / 2}" upper="${PI / 2}"
                effort="${effort}" velocity="${velocity}"/>
     </joint>
-<!-- Link  Support-->
-    <link name="claw_support">
-        <visual>
-            <origin rpy="0 0 ${PI / 2}" xyz="0 -0.05 -0.15"/>
-            <geometry>
-                <mesh filename="package://arm_description/meshes/claw_support.STL" scale="0.01 0.01 0.01"/>
-            </geometry>
-        </visual>
-    </link>
     <joint name ="horizontal_arm_to_claw_support" type="fixed">
         <parent link="horizontal_arm"/>
         <child link = "claw_support"/>
-        <origin xyz="0 0.82 0"/> <!-- Distance image four-->
-    </joint>
-    <!-- Link  gripper -->
-    <link name="gripper_right">
-        <visual>
-            <origin rpy="0 0 -${PI / 2}" xyz="-0.1 0.50 -0.1"/>
-            <geometry>
-                <mesh filename="package://arm_description/meshes/right_finger.STL" scale="0.01 0.01 0.01"/>
-            </geometry>
-        </visual>
-    </link>
-    <link name="gripper_left">
-        <visual>
-            <origin rpy="0 0 -${PI / 2}" xyz="-0.04 0.50 -0.1"/>
-            <geometry>
-                <mesh filename="package://arm_description/meshes/left_finger.STL" scale="0.01 0.01 0.01"/>
-            </geometry>
-        </visual>
-    </link>
+        <origin xyz="0 0.82 0"/>
+    </joint>
     <joint name ="joint_4" type="revolute">
         <parent link="claw_support"/>
         <child link = "gripper_right"/>
-        <origin xyz="-0.04 0.13 -0.1"/> <!-- Distance image five -->
+        <origin xyz="-0.04 0.13 -0.1"/>
         <axis xyz="0 0 1"/>
         <limit lower="-${PI / 2}" upper="0.0"
-        effort="${effort}" velocity="${velocity}"/>
+               effort="${effort}" velocity="${velocity}"/>
     </joint>
     <joint name ="joint_5" type="revolute">
         <parent link="claw_support"/>
         <child link = "gripper_left"/>
-        <origin xyz="-0.22 0.13 -0.1"/> <!-- Distance image five -->
+        <origin xyz="-0.22 0.13 -0.1"/>
         <axis xyz="0 0 1"/>
         <limit lower="0.0" upper="${PI / 2}"
@@ -121,3 +210,8 @@
         <mimic joint="joint_4" multiplier="-1"/>
     </joint>
+    <!-- Transmissions-->
+    <xacro:default_transmission number="1"/>
+    <xacro:default_transmission number="2"/>
+    <xacro:default_transmission number="3"/>
+    <xacro:default_transmission number="4"/>
 </robot>
