Commit message: Configuración

File: arm_ws/src/arm_description/urdf/arm.urdf.xacro (robot description, xacro)
@@ -1,20 +1,6 @@
 <?xml version="1.0"?>
 <robot xmlns:xacro="http://www.ros.org/wiki/xacro" name="arm">
-     <!-- Definir Materiales -->
-  <material name="red">
-    <color rgba="1 0 0 1"/>
-  </material>
-  <material name="blue">
-    <color rgba="0 0 1 1"/>
-  </material>
-  <material name="green">
-    <color rgba="0 1 0 1"/>
-  </material>
-  <material name="yellow">
-    <color rgba="1 1 0 1"/> <!-- Amarillo opaco -->
-  </material>
-  <material name="purple">
-    <color rgba="0.5 0 0.5 1"/> <!-- Púrpura opaco -->
-  </material>
+    <!-- Load Simulated or Real Hardware Interfaces -->
+    <xacro:arg name="is_sim" default="true" />
     <!-- Include Gazebo Parameters -->
     <xacro:include filename="$(find arm_description)/urdf/arm_gazebo.xacro" />
@@ -28,9 +14,9 @@
     <xacro:macro name="default_inertial" params="mass">
         <inertial>
-            <origin xyz="0 0 0" rpy="0 0 0"/>
+            <origin xyz="0 0 0" rpy="0 0 0" />
             <mass value="${mass}" />
             <inertia ixx="1.0" ixy="0.0" ixz="0.0"
-                     iyy="1.0" iyz="0.0"
-                     izz="1.0" />
+                iyy="1.0" iyz="0.0"
+                izz="1.0" />
         </inertial>
     </xacro:macro>
@@ -38,121 +24,151 @@
         <transmission name="transmission_${number}">
             <plugin>transmission_interface/SimpleTransmission</plugin>
-            <actuator name="motor_${number}" role="actuator1"/>
-            <joint name="joint_${number}"    role="joint1">
+            <actuator name="motor_${number}" role="actuator1" />
+            <joint name="joint_${number}" role="joint1">
                 <mechanical_reduction>1.0</mechanical_reduction>
             </joint>
         </transmission>
     </xacro:macro>
+       <!-- Definir Materiales -->
+       <material name="red">
+        <color rgba="1 0 0 1"/>
+      </material>
+      <material name="blue">
+        <color rgba="0 0 1 1"/>
+      </material>
+      <material name="green">
+        <color rgba="0 1 0 1"/>
+      </material>
+      <material name="yellow">
+        <color rgba="1 1 0 1"/> <!-- Amarillo opaco -->
+      </material>
+      <material name="purple">
+        <color rgba="0.5 0 0.5 1"/> <!-- Púrpura opaco -->
+      </material>
     <!-- Links -->
-    <link name="world"/>
+    <link name="world" />
     <link name="base_link">
-        <xacro:default_inertial mass="1.0"/>
-        <visual>
-            <origin rpy="0 0 0" xyz="-0.5 -0.5 0"/>
-            <geometry>
-                <mesh filename="package://arm_description/meshes/basement.STL" scale="0.01 0.01 0.01"/>
-            </geometry>
-            <material name="blue"/>  <!-- Asignar color azul -->
-        </visual>
-        <collision>
-            <origin rpy="0 0 0" xyz="-0.5 -0.5 0"/>
-            <geometry>
-                <mesh filename="package://arm_description/meshes/basement.STL" scale="0.01 0.01 0.01"/>
+        <xacro:default_inertial mass="1.0" />
+        <visual>
+            <origin rpy="0 0 0" xyz="-0.5 -0.5 0" />
+            <geometry>
+                <mesh filename="package://arm_description/meshes/basement.STL"
+                    scale="0.01 0.01 0.01" />
+            </geometry>
+            <material name="blue" />  <!-- Asignar color azul -->
+        </visual>
+        <collision>
+            <origin rpy="0 0 0" xyz="-0.5 -0.5 0" />
+            <geometry>
+                <mesh filename="package://arm_description/meshes/basement.STL"
+                    scale="0.01 0.01 0.01" />
             </geometry>
         </collision>
     </link>
     <link name="base_plate">
-        <xacro:default_inertial mass="0.1"/>
-        <visual>
-            <origin rpy="0 0 0" xyz="-0.39 -0.39 -0.56"/>
-            <geometry>
-                <mesh filename="package://arm_description/meshes/base_plate.STL" scale="0.01 0.01 0.01"/>
-            </geometry>
-            <material name="yellow"/>  <!-- Asignar color azul -->
-        </visual>
-        <collision>
-            <origin rpy="0 0 0" xyz="-0.39 -0.39 -0.56"/>
-            <geometry>
-                <mesh filename="package://arm_description/meshes/base_plate.STL" scale="0.01 0.01 0.01"/>
+        <xacro:default_inertial mass="0.1" />
+        <visual>
+            <origin rpy="0 0 0" xyz="-0.39 -0.39 -0.56" />
+            <geometry>
+                <mesh filename="package://arm_description/meshes/base_plate.STL"
+                    scale="0.01 0.01 0.01" />
+            </geometry>
+            <material name="yellow" />  <!-- Asignar color azul -->
+        </visual>
+        <collision>
+            <origin rpy="0 0 0" xyz="-0.39 -0.39 -0.56" />
+            <geometry>
+                <mesh filename="package://arm_description/meshes/base_plate.STL"
+                    scale="0.01 0.01 0.01" />
             </geometry>
         </collision>
     </link>
     <link name="forward_drive_arm">
-        <xacro:default_inertial mass="0.1"/>
-        <visual>
-            <origin rpy=" 0 -${PI / 2} ${PI / 2}" xyz="0.19 0.06 -0.08"/>
-            <geometry>
-                <mesh filename="package://arm_description/meshes/forward_drive_arm.STL" scale="0.01 0.01 0.01"/>
-            </geometry>
-            <material name="red"/>  <!-- Asignar color azul -->
-        </visual>
-        <collision>
-            <origin rpy=" 0 -${PI / 2} ${PI / 2}" xyz="0.19 0.06 -0.08"/>
-            <geometry>
-                <mesh filename="package://arm_description/meshes/forward_drive_arm.STL" scale="0.01 0.01 0.01"/>
+        <xacro:default_inertial mass="0.1" />
+        <visual>
+            <origin rpy=" 0 -${PI / 2} ${PI / 2}" xyz="0.19 0.06 -0.08" />
+            <geometry>
+                <mesh filename="package://arm_description/meshes/forward_drive_arm.STL"
+                    scale="0.01 0.01 0.01" />
+            </geometry>
+            <material name="red" />  <!-- Asignar color azul -->
+        </visual>
+        <collision>
+            <origin rpy=" 0 -${PI / 2} ${PI / 2}" xyz="0.19 0.06 -0.08" />
+            <geometry>
+                <mesh filename="package://arm_description/meshes/forward_drive_arm.STL"
+                    scale="0.01 0.01 0.01" />
             </geometry>
         </collision>
     </link>
     <link name="horizontal_arm">
-        <xacro:default_inertial mass="0.1"/>
-        <visual>
-            <origin rpy="${PI / 2} 0 ${PI / 2}" xyz="-0.03 -0.4 -0.06"/>
-            <geometry>
-                <mesh filename="package://arm_description/meshes/horizontal_arm.STL" scale="0.01 0.01 0.01"/>
-            </geometry>
-            <material name="red"/>  <!-- Asignar color azul -->
-        </visual>
-        <collision>
-            <origin rpy="${PI / 2} 0 ${PI / 2}" xyz="-0.03 -0.4 -0.06"/>
-            <geometry>
-                <mesh filename="package://arm_description/meshes/horizontal_arm.STL" scale="0.01 0.01 0.01"/>
+        <xacro:default_inertial mass="0.1" />
+        <visual>
+            <origin rpy="${PI / 2} 0 ${PI / 2}" xyz="-0.03 -0.4 -0.06" />
+            <geometry>
+                <mesh filename="package://arm_description/meshes/horizontal_arm.STL"
+                    scale="0.01 0.01 0.01" />
+            </geometry>
+            <material name="red" />  <!-- Asignar color azul -->
+        </visual>
+        <collision>
+            <origin rpy="${PI / 2} 0 ${PI / 2}" xyz="-0.03 -0.4 -0.06" />
+            <geometry>
+                <mesh filename="package://arm_description/meshes/horizontal_arm.STL"
+                    scale="0.01 0.01 0.01" />
             </geometry>
         </collision>
     </link>
     <link name="claw_support">
-        <xacro:default_inertial mass="0.05"/>
-        <visual>
-            <origin rpy="0 0 ${PI / 2}" xyz="0 -0.05 -0.15"/>
-            <geometry>
-                <mesh filename="package://arm_description/meshes/claw_support.STL" scale="0.01 0.01 0.01"/>
-            </geometry>
-            <material name="blue"/>  <!-- Asignar color azul -->
-        </visual>
-        <collision>
-            <origin rpy="0 0 ${PI / 2}" xyz="0 -0.05 -0.15"/>
-            <geometry>
-                <mesh filename="package://arm_description/meshes/claw_support.STL" scale="0.01 0.01 0.01"/>
+        <xacro:default_inertial mass="0.05" />
+        <visual>
+            <origin rpy="0 0 ${PI / 2}" xyz="0 -0.05 -0.15" />
+            <geometry>
+                <mesh filename="package://arm_description/meshes/claw_support.STL"
+                    scale="0.01 0.01 0.01" />
+            </geometry>
+            <material name="blue" />  <!-- Asignar color azul -->
+        </visual>
+        <collision>
+            <origin rpy="0 0 ${PI / 2}" xyz="0 -0.05 -0.15" />
+            <geometry>
+                <mesh filename="package://arm_description/meshes/claw_support.STL"
+                    scale="0.01 0.01 0.01" />
             </geometry>
         </collision>
     </link>
     <link name="gripper_right">
-        <xacro:default_inertial mass="0.01"/>
-        <visual>
-            <origin rpy="0 0 -${PI / 2}" xyz="-0.1 0.50 -0.1"/>
-            <geometry>
-                <mesh filename="package://arm_description/meshes/right_finger.STL" scale="0.01 0.01 0.01"/>
+        <xacro:default_inertial mass="0.01" />
+        <visual>
+            <origin rpy="0 0 -${PI / 2}" xyz="-0.1 0.50 -0.1" />
+            <geometry>
+                <mesh filename="package://arm_description/meshes/right_finger.STL"
+                    scale="0.01 0.01 0.01" />
             </geometry>
             <material name="green"/>  <!-- Asignar color azul -->
         </visual>
         <collision>
-            <origin rpy="0 0 -${PI / 2}" xyz="-0.1 0.50 -0.1"/>
-            <geometry>
-                <mesh filename="package://arm_description/meshes/right_finger.STL" scale="0.01 0.01 0.01"/>
+            <origin rpy="0 0 -${PI / 2}" xyz="-0.1 0.50 -0.1" />
+            <geometry>
+                <mesh filename="package://arm_description/meshes/right_finger.STL"
+                    scale="0.01 0.01 0.01" />
             </geometry>
         </collision>
     </link>
     <link name="gripper_left">
-        <xacro:default_inertial mass="0.01"/>
-        <visual>
-            <origin rpy="0 0 -${PI / 2}" xyz="-0.04 0.50 -0.1"/>
-            <geometry>
-                <mesh filename="package://arm_description/meshes/left_finger.STL" scale="0.01 0.01 0.01"/>
+        <xacro:default_inertial mass="0.01" />
+        <visual>
+            <origin rpy="0 0 -${PI / 2}" xyz="-0.04 0.50 -0.1" />
+            <geometry>
+                <mesh filename="package://arm_description/meshes/left_finger.STL"
+                    scale="0.01 0.01 0.01" />
             </geometry>
             <material name="green"/>  <!-- Asignar color azul -->
         </visual>
         <collision>
-            <origin rpy="0 0 -${PI / 2}" xyz="-0.04 0.50 -0.1"/>
-            <geometry>
-                <mesh filename="package://arm_description/meshes/left_finger.STL" scale="0.01 0.01 0.01"/>
+            <origin rpy="0 0 -${PI / 2}" xyz="-0.04 0.50 -0.1" />
+            <geometry>
+                <mesh filename="package://arm_description/meshes/left_finger.STL"
+                    scale="0.01 0.01 0.01" />
             </geometry>
         </collision>
@@ -160,58 +176,58 @@
     <!-- Joints -->
     <joint name="virtual_joint" type="fixed">
-        <parent link="world"/>
-        <child link="base_link"/>
-        <origin xyz="0 0 0" rpy="0 0 0"/>
-    </joint>
-    <joint name ="joint_1" type="revolute">
-        <parent link="base_link"/>
-        <child link = "base_plate"/>
-        <origin xyz="0 0 0.307"/>
-        <axis xyz="0 0 1"/>
+        <parent link="world" />
+        <child link="base_link" />
+        <origin xyz="0 0 0" rpy="0 0 0" />
+    </joint>
+    <joint name="joint_1" type="revolute">
+        <parent link="base_link" />
+        <child link="base_plate" />
+        <origin xyz="0 0 0.307" />
+        <axis xyz="0 0 1" />
         <limit lower="-${PI / 2}" upper="${PI / 2}"
-               effort="${effort}" velocity="${velocity}"/>
-    </joint>
-    <joint name ="joint_2" type="revolute">
-        <parent link="base_plate"/>
-        <child link = "forward_drive_arm"/>
-        <origin xyz="-0.02 0 0.35"/>
-        <axis xyz="1 0 0"/>
+            effort="${effort}" velocity="${velocity}" />
+    </joint>
+    <joint name="joint_2" type="revolute">
+        <parent link="base_plate" />
+        <child link="forward_drive_arm" />
+        <origin xyz="-0.02 0 0.35" />
+        <axis xyz="1 0 0" />
         <limit lower="-${PI / 2}" upper="${PI / 2}"
-                effort="${effort}" velocity="${velocity}"/>
-    </joint>
-    <joint name ="joint_3" type="revolute">
-        <parent link="forward_drive_arm"/>
-        <child link = "horizontal_arm"/>
-        <origin xyz="0 0 0.8"/>
-        <axis xyz="1 0 0"/>
+            effort="${effort}" velocity="${velocity}" />
+    </joint>
+    <joint name="joint_3" type="revolute">
+        <parent link="forward_drive_arm" />
+        <child link="horizontal_arm" />
+        <origin xyz="0 0 0.8" />
+        <axis xyz="1 0 0" />
         <limit lower="-${PI / 2}" upper="${PI / 2}"
-               effort="${effort}" velocity="${velocity}"/>
-    </joint>
-    <joint name ="horizontal_arm_to_claw_support" type="fixed">
-        <parent link="horizontal_arm"/>
-        <child link = "claw_support"/>
-        <origin xyz="0 0.82 0"/>
-    </joint>
-    <joint name ="joint_4" type="revolute">
-        <parent link="claw_support"/>
-        <child link = "gripper_right"/>
-        <origin xyz="-0.04 0.13 -0.1"/>
-        <axis xyz="0 0 1"/>
+            effort="${effort}" velocity="${velocity}" />
+    </joint>
+    <joint name="horizontal_arm_to_claw_support" type="fixed">
+        <parent link="horizontal_arm" />
+        <child link="claw_support" />
+        <origin xyz="0 0.82 0" />
+    </joint>
+    <joint name="joint_4" type="revolute">
+        <parent link="claw_support" />
+        <child link="gripper_right" />
+        <origin xyz="-0.04 0.13 -0.1" />
+        <axis xyz="0 0 1" />
         <limit lower="-${PI / 2}" upper="0.0"
-               effort="${effort}" velocity="${velocity}"/>
-    </joint>
-    <joint name ="joint_5" type="revolute">
-        <parent link="claw_support"/>
-        <child link = "gripper_left"/>
-        <origin xyz="-0.22 0.13 -0.1"/>
-        <axis xyz="0 0 1"/>
+            effort="${effort}" velocity="${velocity}" />
+    </joint>
+    <joint name="joint_5" type="revolute">
+        <parent link="claw_support" />
+        <child link="gripper_left" />
+        <origin xyz="-0.22 0.13 -0.1" />
+        <axis xyz="0 0 1" />
         <limit lower="0.0" upper="${PI / 2}"
-               effort="${effort}" velocity="${velocity}"/>
-        <mimic joint="joint_4" multiplier="-1"/>
+            effort="${effort}" velocity="${velocity}" />
+        <mimic joint="joint_4" multiplier="-1" />
     </joint>
     <!-- Transmissions-->
-    <xacro:default_transmission number="1"/>
-    <xacro:default_transmission number="2"/>
-    <xacro:default_transmission number="3"/>
-    <xacro:default_transmission number="4"/>
+    <xacro:default_transmission number="1" />
+    <xacro:default_transmission number="2" />
+    <xacro:default_transmission number="3" />
+    <xacro:default_transmission number="4" />
 </robot>

File: arm_ws/src/arm_description/urdf/arm_gazebo.xacro (robot description, xacro)
@@ -1,32 +1,32 @@
 <?xml version="1.0"?>
 <robot xmlns:xacro="http://www.ros.org/wiki/xacro" name="arm">
-   <gazebo reference = "base_link">
+  <gazebo reference="base_link">
     <material>Gazebo/Blue</material>
   </gazebo>
-  <gazebo reference = "base_plate">
+  <gazebo reference="base_plate">
     <material>Gazebo/Yellow</material>
   </gazebo>
-  <gazebo reference = "forward_drive_arm">
+  <gazebo reference="forward_drive_arm">
     <material>Gazebo/Red</material>
   </gazebo>
-  <gazebo reference = "horizontal_arm">
+  <gazebo reference="horizontal_arm">
     <material>Gazebo/Red</material>
   </gazebo>
-  <gazebo reference = "claw_support">
+  <gazebo reference="claw_support">
     <material>Gazebo/Blue</material>
   </gazebo>
-  <gazebo reference = "gripper_right">
+  <gazebo reference="gripper_right">
     <material>Gazebo/Green</material>
   </gazebo>
-  <gazebo reference = "gripper_left">
+  <gazebo reference="gripper_left">
     <material>Gazebo/Green</material>
   </gazebo>
-    <!-- Gazebo ros2_control plugin -->
-    <gazebo>
-      <plugin filename="libgazebo_ros2_control.so" name="gazebo_ros2_control">
-        <robot_param>robot_description</robot_param>
-        <robot_param_node>robot_state_publisher</robot_param_node>
-        <parameters>$(find arm_controller)/config/arm_controllers.yaml</parameters>
-      </plugin>
-    </gazebo>
+  <!-- Gazebo ros2_control plugin -->
+  <gazebo>
+    <plugin filename="libgazebo_ros2_control.so" name="gazebo_ros2_control">
+      <robot_param>robot_description</robot_param>
+      <robot_param_node>robot_state_publisher</robot_param_node>
+      <parameters>$(find arm_controller)/config/arm_controllers.yaml</parameters>
+    </plugin>
+  </gazebo>
 </robot>

File: arm_ws/src/arm_description/urdf/arm_ros2_control.xacro (robot description, xacro)
@@ -4,7 +4,24 @@
         <xacro:property name="PI" value="3.14159265359" />
         <!-- ros2_control Gazebo -->
-        <hardware>
-            <plugin>gazebo_ros2_control/GazeboSystem</plugin>
-        </hardware>
+        <xacro:if value="$(arg is_sim)">
+            <hardware>
+                <plugin>gazebo_ros2_control/GazeboSystem</plugin>
+            </hardware>
+            <joint name="joint_5">
+                <param name="mimic">joint_4</param>
+                <param name="multiplier">-1</param>
+                <command_interface name="position">
+                <param name="min">0.0</param>
+                <param name="max">${PI / 2}</param>
+                </command_interface>
+            </joint>
+        </xacro:if>
+        <!-- ros2_control Real Robot -->
+        <xacro:unless value="$(arg is_sim)">
+            <hardware>
+                <plugin>arm_controller/armInterface</plugin>
+                <param name="port">/dev/ttyACM0</param>
+            </hardware>
+        </xacro:unless>
         <joint name="joint_1">
             <command_interface name="position">
@@ -35,12 +52,4 @@
             <state_interface name="position"/>
         </joint>
-        <joint name="joint_5">
-            <param name="mimic">joint_4</param>
-            <param name="multiplier">-1</param>
-            <command_interface name="position">
-            <param name="min">0.0</param>
-            <param name="max">${PI / 2}</param>
-            </command_interface>
-        </joint>
     </ros2_control>
 </robot>
